Commit message: Adding gazebo simulation files.

File: robots/KR5sixxR650WP_gazebo.URDF (robot description, URDF)
Before this commit: robot KR5sixxR650WP_description, 7 links, 6 joints
Links:
- added link world
Joints:
- added joint fixed: type fixed, parent world, child base_link
- joint elbow_pitch: limit lower=-3.647738137 upper=0.959931089 effort=4 velocity=6.545 -> lower=-3.647738137 upper=0.959931089 effort=330 velocity=6.545
- joint elbow_roll: limit lower=-3.3161 upper=3.3161 effort=2 velocity=7.1558 -> lower=-3.3161 upper=3.3161 effort=550 velocity=7.1558
- joint shoulder_pitch: limit lower=-1.745329252 upper=2.35619449 effort=4 velocity=5.236 -> lower=-1.745329252 upper=2.35619449 effort=330 velocity=5.236
- joint shoulder_yaw: limit lower=-2.9671 upper=2.9671 effort=4 velocity=6.545 -> lower=-2.9671 upper=2.9671 effort=330 velocity=6.545
- joint wrist_pitch: limit lower=-2.094395102 upper=2.094395102 effort=2 velocity=7.1558 -> lower=-2.094395102 upper=2.094395102 effort=54 velocity=7.1558
- joint wrist_roll: limit lower=-6.24827872 upper=6.24827872 effort=2 velocity=11.5191731 -> lower=-6.24827872 upper=6.24827872 effort=54 velocity=11.5191731
