Commit message: Fixed joint limits.

File: robots/KR5sixxR650WP_description.URDF (robot description, URDF)
Before this commit: robot KR5sixxR650WP_description, 7 links, 6 joints
Joints:
- joint elbow_pitch: limit lower=-2.0769 upper=2.8798 effort=0 velocity=6.545 -> lower=-3.647738137 upper=0.959931089 effort=0 velocity=6.545
- joint shoulder_pitch: limit lower=-3.3161 upper=0.7854 effort=0 velocity=5.236 -> lower=-1.745329252 upper=2.35619449 effort=0 velocity=5.236
- joint wrist_pitch: limit lower=-2.0944 upper=2.0944 effort=0 velocity=7.1558 -> lower=-2.094395102 upper=2.094395102 effort=0 velocity=7.1558

Commit message: Adding tool changer in GTRI configuration.

File: robots/KR5sixxR650WP_description.URDF (robot description, URDF)
Before this commit: robot KR5sixxR650WP_description, 7 links, 6 joints
Links:
- added link tool_changer_link, mass 0.0809599830898989; collision mesh filename=package://KR5sixxR650WP_description/meshes/tool_changer_lin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; visual mesh filename=package://KR5sixxR650WP_description/meshes/tool_changer_lin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
Joints:
- added joint tool_changer_offset: type fixed, parent palm, child tool_changer_link, origin xyz=0.063701 0 0 rpy=0 0 0, axis 0 0 0
- joint elbow_pitch: limit lower=-3.647738137 upper=0.959931089 effort=0 velocity=6.545 -> lower=-3.647738137 upper=0.959931089 effort=2 velocity=6.545
- joint elbow_roll: limit lower=-3.3161 upper=3.3161 effort=0 velocity=7.1558 -> lower=-3.3161 upper=3.3161 effort=2 velocity=7.1558
- joint shoulder_pitch: limit lower=-1.745329252 upper=2.35619449 effort=0 velocity=5.236 -> lower=-1.745329252 upper=2.35619449 effort=2 velocity=5.236
- joint shoulder_yaw: limit lower=-2.9671 upper=2.9671 effort=0 velocity=6.545 -> lower=-2.9671 upper=2.9671 effort=2 velocity=6.545
- joint wrist_pitch: limit lower=-2.094395102 upper=2.094395102 effort=0 velocity=7.1558 -> lower=-2.094395102 upper=2.094395102 effort=2 velocity=7.1558
- joint wrist_roll: limit lower=-6.24827872 upper=6.24827872 effort=0 velocity=11.5191731 -> lower=-6.24827872 upper=6.24827872 effort=2 velocity=11.5191731

Commit message: Aligned EE frame with tool changer.

File: robots/KR5sixxR650WP_description.URDF (robot description, URDF)
Before this commit: robot KR5sixxR650WP_description, 8 links, 7 joints
Links:
- link base_link: mass 7.58585707666653 -> None
Joints:
- joint tool_changer_offset: origin xyz=0.063701 0 0 rpy=0 0 0 -> xyz=0.063700999999999 0 0 rpy=-0.392684216336714 0 0

Commit message: Added collision meshes.

File: robots/KR5sixxR650WP_description.URDF (robot description, URDF)
Before this commit: robot KR5sixxR650WP_description, 7 links, 6 joints
Links:
- link base_link: geometry collision mesh filename=package://KR5sixxR650WP_description/meshes/base_link_collis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; visual mesh filename=package://KR5sixxR650WP_description/meshes/base_link.STL
- link bicep: geometry collision mesh filename=package://KR5sixxR650WP_description/meshes/bicep_collision.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; visual mesh filename=package://KR5sixxR650WP_description/meshes/bicep.STL
- link elbow: geometry collision mesh filename=package://KR5sixxR650WP_description/meshes/elbow_collision.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; visual mesh filename=package://KR5sixxR650WP_description/meshes/elbow.STL
- link forearm: geometry collision mesh filename=package://KR5sixxR650WP_description/meshes/forearm_collisio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; visual mesh filename=package://KR5sixxR650WP_description/meshes/forearm.STL
- link palm: geometry collision mesh filename=package://KR5sixxR650WP_description/meshes/palm_collision.S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; visual mesh filename=package://KR5sixxR650WP_description/meshes/palm.STL
- link shoulder: geometry collision mesh filename=package://KR5sixxR650WP_description/meshes/shoulder_collisi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; visual mesh filename=package://KR5sixxR650WP_description/meshes/shoulder.STL
- link wrist: geometry collision mesh filename=package://KR5sixxR650WP_description/meshes/wrist_collision.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; visual mesh filename=package://KR5sixxR650WP_description/meshes/wrist.STL

Commit message: Removed inertia tag from base link.

File: robots/KR5sixxR650WP_description.URDF (robot description, URDF)
Before this commit: robot KR5sixxR650WP_description, 7 links, 6 joints
Links:
- link base_link: mass 7.58585707666653 -> None
